File: MBARETECH.kicad_pcb (KiCad board)
At the start: 2 copper layers, 100 x 100 mm, 53 parts, among them SW1 SW1, SW2 SW2, U1 ESP32-S3-DEVKITC-1-N8R2

Commit message: final
Parts:
- R16: value 10k -> R16
- R17: value 10k -> R17
- R18: value 10k -> R18
- R19: value 10k -> R19
Connections:
- ? pad 1: GND -> -BATT (x4)
